Commit message: updated sdf model to new robot design

File: sdf/robot.xacro (robot description, xacro)
@@ -2,5 +2,5 @@
     <xacro:property name="base_friction" value="0.75"/>
     <xacro:property name="arm_friction" value="0.28"/>
-    <xacro:property name="servo_height" value="0.043"/>
+    <xacro:property name="servo_height" value="0.032"/>
     <xacro:property name="draft_angle" value="-0.349066"/>
     <xacro:property name="_120_degrees" value="2.0944"/>
@@ -26,5 +26,5 @@
             <inertial> <!--inertial properties of the link mass, inertia matix-->
                 <mass>0.123</mass>
-                <pose>0 0 0.022 0 0 0</pose>
+                <pose>0 0 0.019 0 0 0</pose>
                 <inertia>
                     <ixx>0.00015</ixx>
@@ -37,9 +37,9 @@
             </inertial>
             <visual name='visual'>
-                <pose>0 0 0.025 0 0 0</pose>
+                <pose>0 0 0.019 0 0 0</pose>
                 <geometry>
                     <cylinder>
                         <radius>0.050</radius>
-                        <length>0.050</length>
+                        <length>0.038</length>
                     </cylinder>
                 </geometry>
@@ -113,10 +113,10 @@
             </joint>
         </xacro:macro>
-        <xacro:base_collision_macro number='1' x='-0.085'   y='0.010'   radius='0.004'/>
-        <xacro:base_collision_macro number='2' x='0.034'    y='0.079'   radius='0.004'/>
-        <xacro:base_collision_macro number='3' x='0.051'    y='0.069'   radius='0.004'/>
-        <xacro:base_collision_macro number='4' x='0.051'    y='-0.069'  radius='0.004'/>
-        <xacro:base_collision_macro number='5' x='0.034'    y='-0.079'  radius='0.004'/>
-        <xacro:base_collision_macro number='6' x='-0.085'   y='-0.010'  radius='0.004'/>
+        <xacro:base_collision_macro number='1' x='-0.081'   y='0.008'   radius='0.004'/>
+        <xacro:base_collision_macro number='2' x='0.033'    y='0.074'   radius='0.004'/>
+        <xacro:base_collision_macro number='3' x='0.0475'    y='0.066'   radius='0.004'/>
+        <xacro:base_collision_macro number='4' x='0.0475'    y='-0.066'  radius='0.004'/>
+        <xacro:base_collision_macro number='5' x='0.033'    y='-0.074'  radius='0.004'/>
+        <xacro:base_collision_macro number='6' x='-0.081'   y='-0.008'  radius='0.004'/>
         <xacro:macro name='servo_macro' params='number x y roll yaw '>
             <link name='servo${number}_link'>
@@ -181,12 +181,12 @@
                     <geometry>
                         <cylinder>
-                            <radius>0.0050</radius>
+                            <radius>0.0030</radius>
                             <length>${arm_length}</length>
                         </cylinder>
                     </geometry>
                     <material>
-                        <ambient>1.0 0.0 1.0 1</ambient>
-                        <diffuse>1.0 0.0 1.0 1</diffuse>
-                        <specular>1.0 0.0 1.0 1</specular>
+                        <ambient>0.0 0.0 1.0 1</ambient>
+                        <diffuse>0.0 0.0 1.0 1</diffuse>
+                        <specular>0.0 0.0 1.0 1</specular>
                     </material>
                 </visual>
@@ -223,5 +223,5 @@
                 <inertial>
                     <mass>0.001</mass>
-                    <pose>0 ${arm_length} 0 0 0 0</pose>
+                    <pose>0 ${arm_length + 0.002}  0 0 0 0</pose>
                     <inertia>
                         <ixx>0.0000041</ixx>
@@ -234,5 +234,5 @@
                 </inertial>
                 <visual name='visual'>
-                    <pose>0 ${arm_length} 0 0 0 0</pose>
+                    <pose>0 ${arm_length + 0.002} 0 0 0 0</pose>
                     <geometry>
                         <sphere>
@@ -247,5 +247,5 @@
                 </visual>
                 <collision name='collision'>
-                    <pose>0 ${arm_length} 0 0 0 0</pose>
+                    <pose>0 ${arm_length + 0.002} 0 0 0 0</pose>
                     <geometry>
                         <sphere>

Commit message: small collision spheres

File: sdf/robot.xacro (robot description, xacro)
@@ -2,5 +2,5 @@
     <xacro:property name="base_friction" value="0.75"/>
     <xacro:property name="arm_friction" value="0.28"/>
-    <xacro:property name="servo_height" value="0.032"/>
+    <xacro:property name="servo_height" value="0.028"/>
     <xacro:property name="draft_angle" value="-0.349066"/>
     <xacro:property name="_120_degrees" value="2.0944"/>
@@ -113,10 +113,10 @@
             </joint>
         </xacro:macro>
-        <xacro:base_collision_macro number='1' x='-0.081'   y='0.008'   radius='0.004'/>
-        <xacro:base_collision_macro number='2' x='0.033'    y='0.074'   radius='0.004'/>
-        <xacro:base_collision_macro number='3' x='0.0475'    y='0.066'   radius='0.004'/>
-        <xacro:base_collision_macro number='4' x='0.0475'    y='-0.066'  radius='0.004'/>
-        <xacro:base_collision_macro number='5' x='0.033'    y='-0.074'  radius='0.004'/>
-        <xacro:base_collision_macro number='6' x='-0.081'   y='-0.008'  radius='0.004'/>
+        <xacro:base_collision_macro number='1' x='-0.081'   y='0.008'   radius='0.0025'/>
+        <xacro:base_collision_macro number='2' x='0.033'    y='0.074'   radius='0.0025'/>
+        <xacro:base_collision_macro number='3' x='0.0475'    y='0.066'   radius='0.0025'/>
+        <xacro:base_collision_macro number='4' x='0.0475'    y='-0.066'  radius='0.0025'/>
+        <xacro:base_collision_macro number='5' x='0.033'    y='-0.074'  radius='0.0025'/>
+        <xacro:base_collision_macro number='6' x='-0.081'   y='-0.008'  radius='0.0025'/>
         <xacro:macro name='servo_macro' params='number x y roll yaw '>
             <link name='servo${number}_link'>
@@ -237,5 +237,5 @@
                     <geometry>
                         <sphere>
-                            <radius>0.0060</radius>
+                            <radius>0.0025</radius>
                         </sphere>
                     </geometry>
@@ -250,5 +250,5 @@
                     <geometry>
                         <sphere>
-                            <radius>0.0060</radius>
+                            <radius>0.0025</radius>
                         </sphere>
                     </geometry>

Commit message: more accurate collisions

File: sdf/robot.xacro (robot description, xacro)
@@ -2,5 +2,5 @@
     <xacro:property name="base_friction" value="0.75"/>
     <xacro:property name="arm_friction" value="0.28"/>
-    <xacro:property name="servo_height" value="0.028"/>
+    <xacro:property name="servo_height" value="0.033"/>
     <xacro:property name="draft_angle" value="-0.349066"/>
     <xacro:property name="_120_degrees" value="2.0944"/>
@@ -219,53 +219,4 @@
                 </axis>
             </joint>
-            <link name='arm${number}_end_link'>
-                <pose relative_to='arm${number}_link'/>
-                <inertial>
-                    <mass>0.001</mass>
-                    <pose>0 ${arm_length + 0.002}  0 0 0 0</pose>
-                    <inertia>
-                        <ixx>0.0000041</ixx>
-                        <ixy>0</ixy>
-                        <ixz>0</ixz>
-                        <iyy>0.00000033</iyy>
-                        <iyz>0</iyz>
-                        <izz>0.0000039</izz>
-                    </inertia>
-                </inertial>
-                <visual name='visual'>
-                    <pose>0 ${arm_length + 0.002} 0 0 0 0</pose>
-                    <geometry>
-                        <sphere>
-                            <radius>0.0025</radius>
-                        </sphere>
-                    </geometry>
-                    <material>
-                        <ambient>1.0 0.0 1.0 1</ambient>
-                        <diffuse>1.0 0.0 1.0 1</diffuse>
-                        <specular>1.0 0.0 1.0 1</specular>
-                    </material>
-                </visual>
-                <collision name='collision'>
-                    <pose>0 ${arm_length + 0.002} 0 0 0 0</pose>
-                    <geometry>
-                        <sphere>
-                            <radius>0.0025</radius>
-                        </sphere>
-                    </geometry>
-                    <surface>
-                        <friction>
-                            <ode>
-                            <mu>${arm_friction}</mu>
-                            <mu2>${arm_friction}</mu2>
-                            </ode>
-                        </friction>
-                    </surface>
-                </collision>
-            </link>
-            <joint name='arm${number}_end_joint' type='fixed'>
-                <pose relative_to='arm${number}_end_link'/>
-                <parent>arm${number}_link</parent>
-                <child>arm${number}_end_link</child>
-            </joint>
             <plugin
                 filename="libignition-gazebo-joint-position-controller-system.so"
@@ -284,4 +235,61 @@
         <xacro:servo_macro number='5' x='${servo5_x}' y='${servo5_y}'  roll='0'                 yaw='${_240_degrees}'/>
         <xacro:servo_macro number='6' x='${servo6_x}' y='${servo6_y}'  roll='${_180_degrees}'   yaw='${_240_degrees}'/>
+        <xacro:macro name='arm_collision_macro' params='number radius z_offset'>
+            <link name='arm${number}_end_link'>
+                <pose relative_to='arm${number}_link'> -0.0033 ${arm_length + 0.0032} ${z_offset} 0 0 0 </pose>
+                <inertial>
+                    <mass>0.001</mass>
+                    <pose>0 0 0 0 0 0</pose>
+                    <inertia>
+                        <ixx>0.0000041</ixx>
+                        <ixy>0</ixy>
+                        <ixz>0</ixz>
+                        <iyy>0.00000033</iyy>
+                        <iyz>0</iyz>
+                        <izz>0.0000039</izz>
+                    </inertia>
+                </inertial>
+                <visual name='visual'>
+                    <pose>0 0 0 0 0 0</pose>
+                    <geometry>
+                        <sphere>
+                            <radius>0.0025</radius>
+                        </sphere>
+                    </geometry>
+                    <material>
+                        <ambient>1.0 0.0 1.0 1</ambient>
+                        <diffuse>1.0 0.0 1.0 1</diffuse>
+                        <specular>1.0 0.0 1.0 1</specular>
+                    </material>
+                </visual>
+                <collision name='collision'>
+                    <pose>0 0 0 0 0 0</pose>
+                    <geometry>
+                        <sphere>
+                            <radius>0.0025</radius>
+                        </sphere>
+                    </geometry>
+                    <surface>
+                        <friction>
+                            <ode>
+                            <mu>${arm_friction}</mu>
+                            <mu2>${arm_friction}</mu2>
+                            </ode>
+                        </friction>
+                    </surface>
+                </collision>
+            </link>
+            <joint name='arm${number}_end_joint' type='fixed'>
+                <pose relative_to='arm${number}_end_link'/>
+                <parent>arm${number}_link</parent>
+                <child>arm${number}_end_link</child>
+            </joint>
+        </xacro:macro>
+        <xacro:arm_collision_macro number='1' radius='0.0025' z_offset='-0.0063'/>
+        <xacro:arm_collision_macro number='2' radius='0.0025' z_offset='0.0063'/>
+        <xacro:arm_collision_macro number='3' radius='0.0025' z_offset='-0.0063'/>
+        <xacro:arm_collision_macro number='4' radius='0.0025' z_offset='0.0063'/>
+        <xacro:arm_collision_macro number='5' radius='0.0025' z_offset='-0.0063'/>
+        <xacro:arm_collision_macro number='6' radius='0.0025' z_offset='0.0063'/>
         <plugin filename="libignition-gazebo-pose-publisher-system.so" name="ignition::gazebo::systems::PosePublisher">
             <publish_nested_model_pose>true</publish_nested_model_pose>

File: sdf/world.xacro (robot description, xacro)
@@ -2,5 +2,5 @@
         <physics name="1ms" type="ignored">
             <max_step_size>0.005</max_step_size>
-            <real_time_factor>10.0</real_time_factor>
+            <real_time_factor>1.0</real_time_factor>
         </physics>
         <plugin
